File: IO Board.kicad_pcb (KiCad board)
At the start: 2 copper layers, 32 x 63.5 mm, 10 parts, among them J1 DM3AT-SF-PEJM5, J2 2x20-pin_TRS-20_bus, U1 DS3232M, U2 SN74LVC1G07DBVR

Commit message: check twice, fab once
Routing:
- net Net-(BT1-Pad1): track 28.7 -> 45.8 mm
- net GNDREF: track 26.2 -> 19.2 mm, vias 7 -> 6
Other:
- rule pad_to_mask_clearance: 0 -> 0.1
- board text added: "I/O board rev B"
- board text removed: "I/O board rev A"
Changed lines of the file:
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@@
     (thickness 1.6)
     (drawings 10)
-    (tracks 107)
+    (tracks 109)
     (zones 0)
     (modules 10)
@@
     (pad_size 1.524 1.524)
     (pad_drill 0.762)
-    (pad_to_mask_clearance 0)
+    (pad_to_mask_clearance 0.1)
     (solder_mask_min_width 0.2)
     (aux_axis_origin 0 0)
@@
     (add_net "Net-(U1-Pad3)")
     (add_net "Net-(U2-Pad1)")
+  )
+  (module "cpu board:Keystone-3002TR-0" (layer F.Cu)
+    (at 160.2105 -41.148 270)
+    (fp_text reference BT1 (at -12.827 3.4925 180) (layer F.SilkS)
+      (effects (font (size 1 1) (thickness 0.15)) (justify right))
+    )
+    (fp_text value "Keystone 3002" (at 3.556 0.381 180) (layer F.SilkS)
+      (effects (font (size 1.27 1.27) (thickness 0.15)))
+    )
+    (fp_line (start -10.555 9.93) (end -10.555 -9.93) (layer F.Fab) (width 0.15))
+    (fp_line (start -10.555 -9.93) (end 10.555 -9.93) (layer F.Fab) (width 0.15))
+    (fp_line (start 10.555 -9.93) (end 10.555 9.93) (layer F.Fab) (width 0.15))
+    (fp_line (start 10.555 9.93) (end -10.555 9.93) (layer F.Fab) (width 0.15))
+    (fp_line (start 10.555 -9.93) (end -10.555 -9.93) (layer F.SilkS) (width 0.15))
+    (fp_line (start 10.555 9.93) (end -10.555 9.93) (layer F.SilkS) (width 0.15))
+    (fp_line (start 10.555 -9.925) (end 10.555 -3.025) (layer F.SilkS) (width 0.15))
+    (fp_line (start -10.555 -9.925) (end -10.555 -3.025) (layer F.SilkS) (width 0.15))
+    (fp_line (start 10.555 3.025) (end 10.555 9.925) (layer F.SilkS) (width 0.15))
+    (fp_line (start -10.555 3.025) (end -10.555 9.925) (layer F.SilkS) (width 0.15))
+    (fp_line (start 15.39 -9.98) (end 15.39 -9.98) (layer F.CrtYd) (width 0.15))
+    (fp_line (start 15.39 -9.98) (end -15.39 -9.98) (layer F.CrtYd) (width 0.15))
+    (fp_line (start -15.39 -9.98) (end -15.39 9.98) (layer F.CrtYd) (width 0.15))
+    (fp_line (start -15.39 9.98) (end 15.39 9.98) (layer F.CrtYd) (width 0.15))
+    (fp_line (start 15.39 9.98) (end 15.39 -9.98) (layer F.CrtYd) (width 0.15))
+    (fp_circle (center 0.135 -10.55) (end 0.26 -10.55) (layer F.SilkS) (width 0.25))
+    (pad 2 smd rect (at 0 0 270) (size 3.96 3.96) (layers F.Cu F.Paste F.Mask)
+      (net 41 GNDREF))
+    (pad 1 smd rect (at -12.825 0 270) (size 5.08 5.08) (layers F.Cu F.Paste F.Mask)
+      (net 1 "Net-(BT1-Pad1)"))
+    (pad 1 smd rect (at 12.825 0 270) (size 5.08 5.08) (layers F.Cu F.Paste F.Mask)
+      (net 1 "Net-(BT1-Pad1)"))
+    (model eec.models/Keystone_-_3002TR.step
+      (at (xyz 0 0 0))
+      (scale (xyz 1 1 1))
+      (rotate (xyz 0 0 0))
+    )
+    (model ${KIPRJMOD}/Keystone_-_3002TR.step
+      (at (xyz 0 0 0))
+      (scale (xyz 1 1 1))
+      (rotate (xyz 0 0 0))
+    )
   )
   (module Connector_PinHeader_2.54mm:PinHeader_2x20_P2.54mm_Vertical (layer F.Cu)
@@
     )
   )
-  (module "cpu board:Keystone-3002TR-0" (layer F.Cu)
-    (at 160.2105 -41.148 270)
-    (fp_text reference BT1 (at -12.827 3.4925 180) (layer F.SilkS)
-      (effects (font (size 1 1) (thickness 0.15)) (justify right))
-    )
-    (fp_text value "Keystone 3002" (at 3.556 0.381 180) (layer F.SilkS)
-      (effects (font (size 1.27 1.27) (thickness 0.15)))
-    )
-    (fp_line (start -10.555 9.93) (end -10.555 -9.93) (layer F.Fab) (width 0.15))
-    (fp_line (start -10.555 -9.93) (end 10.555 -9.93) (layer F.Fab) (width 0.15))
-    (fp_line (start 10.555 -9.93) (end 10.555 9.93) (layer F.Fab) (width 0.15))
-    (fp_line (start 10.555 9.93) (end -10.555 9.93) (layer F.Fab) (width 0.15))
-    (fp_line (start 10.555 -9.93) (end -10.555 -9.93) (layer F.SilkS) (width 0.15))
-    (fp_line (start 10.555 9.93) (end -10.555 9.93) (layer F.SilkS) (width 0.15))
-    (fp_line (start 10.555 -9.925) (end 10.555 -3.025) (layer F.SilkS) (width 0.15))
-    (fp_line (start -10.555 -9.925) (end -10.555 -3.025) (layer F.SilkS) (width 0.15))
-    (fp_line (start 10.555 3.025) (end 10.555 9.925) (layer F.SilkS) (width 0.15))
-    (fp_line (start -10.555 3.025) (end -10.555 9.925) (layer F.SilkS) (width 0.15))
-    (fp_line (start 15.39 -9.98) (end 15.39 -9.98) (layer F.CrtYd) (width 0.15))
-    (fp_line (start 15.39 -9.98) (end -15.39 -9.98) (layer F.CrtYd) (width 0.15))
-    (fp_line (start -15.39 -9.98) (end -15.39 9.98) (layer F.CrtYd) (width 0.15))
-    (fp_line (start -15.39 9.98) (end 15.39 9.98) (layer F.CrtYd) (width 0.15))
-    (fp_line (start 15.39 9.98) (end 15.39 -9.98) (layer F.CrtYd) (width 0.15))
-    (fp_circle (center 0.135 -10.55) (end 0.26 -10.55) (layer F.SilkS) (width 0.25))
-    (pad 1 smd rect (at 0 0 270) (size 3.96 3.96) (layers F.Cu F.Paste F.Mask)
-      (net 1 "Net-(BT1-Pad1)"))
-    (pad 2 smd rect (at -12.825 0 270) (size 5.08 5.08) (layers F.Cu F.Paste F.Mask)
-      (net 41 GNDREF))
-    (pad 2 smd rect (at 12.825 0 270) (size 5.08 5.08) (layers F.Cu F.Paste F.Mask)
-      (net 41 GNDREF))
-    (model eec.models/Keystone_-_3002TR.step
-      (at (xyz 0 0 0))
-      (scale (xyz 1 1 1))
-      (rotate (xyz 0 0 0))
-    )
-    (model ${KIPRJMOD}/Keystone_-_3002TR.step
-      (at (xyz 0 0 0))
-      (scale (xyz 1 1 1))
-      (rotate (xyz 0 0 0))
-    )
-  )
   (gr_text JLCJLCJLCJLC (at 159.3215 -70.0405) (layer F.SilkS)
     (effects (font (size 1 1) (thickness 0.25)))
   )
-  (gr_text "I/O board rev A" (at 160.2105 -23.749) (layer F.SilkS)
+  (gr_text "I/O board rev B" (at 160.2105 -23.749) (layer F.SilkS)
     (effects (font (size 1.5 1.5) (thickness 0.3)))
   )
@@
   (gr_arc (start 151.511 -82.55) (end 151.511 -85.09) (angle -90) (layer Edge.Cuts) (width 0.15))
   (gr_arc (start 178.435 -82.55) (end 180.975 -82.55) (angle -90) (layer Edge.Cuts) (width 0.15))
-  (segment (start 152.104 -62.738) (end 150.368 -61.002) (width 0.25) (layer F.Cu) (net 1))
+  (segment (start 160.2105 -31.113) (end 154.9908 -36.3327) (width 0.25) (layer F.Cu) (net 1))
+  (segment (start 160.2105 -28.323) (end 160.2105 -31.113) (width 0.25) (layer F.Cu) (net 1))
+  (segment (start 154.9908 -36.3327) (end 154.9908 -42.8752) (width 0.25) (layer F.Cu) (net 1))
+  (segment (start 160.2105 -48.0949) (end 160.2105 -53.973) (width 0.25) (layer F.Cu) (net 1))
+  (segment (start 154.9908 -42.8752) (end 160.2105 -48.0949) (width 0.25) (layer F.Cu) (net 1))
+  (segment (start 152.104 -62.738) (end 150.876 -61.51) (width 0.25) (layer F.Cu) (net 1))
   (segment (start 153.129 -62.738) (end 152.104 -62.738) (width 0.25) (layer F.Cu) (net 1))
-  (segment (start 157.9805 -41.148) (end 160.2105 -41.148) (width 0.25) (layer F.Cu) (net 1))
-  (segment (start 150.368 -48.7605) (end 157.9805 -41.148) (width 0.25) (layer F.Cu) (net 1))
-  (segment (start 150.368 -61.002) (end 150.368 -48.7605) (width 0.25) (layer F.Cu) (net 1))
+  (segment (start 157.4205 -53.973) (end 160.2105 -53.973) (width 0.25) (layer F.Cu) (net 1))
+  (segment (start 150.876 -60.5175) (end 157.4205 -53.973) (width 0.25) (layer F.Cu) (net 1))
+  (segment (start 150.876 -61.51) (end 150.876 -60.5175) (width 0.25) (layer F.Cu) (net 1))
   (segment (start 173.576999 -59.778001) (end 170.41 -62.945) (width 0.25) (layer F.Cu) (net 5))
   (segment (start 170.41 -62.945) (end 169.86 -62.945) (width 0.25) (layer F.Cu) (net 5))
@@
   (segment (start 166.2075 -64.897) (end 166.2075 -61.877) (width 0.25) (layer F.Cu) (net 41))
   (segment (start 163.943 -61.468) (end 165.7985 -61.468) (width 0.25) (layer F.Cu) (net 41))
-  (via (at 166.116 -53.975) (size 0.8) (drill 0.4) (layers F.Cu B.Cu) (net 41))
-  (via (at 166.1775 -28.323) (size 0.8) (drill 0.4) (layers F.Cu B.Cu) (net 41))
   (via (at 150.622 -64.008) (size 0.8) (drill 0.4) (layers F.Cu B.Cu) (net 41))
   (segment (start 153.129 -64.008) (end 150.622 -64.008) (width 0.25) (layer F.Cu) (net 41))
@@
   (via (at 172.72 -75.819) (size 0.8) (drill 0.4) (layers F.Cu B.Cu) (net 41))
   (segment (start 171.069 -75.819) (end 172.72 -75.819) (width 0.25) (layer F.Cu) (net 41))
-  (segment (start 163.0005 -28.323) (end 166.1775 -28.323) (width 0.25) (layer F.Cu) (net 41))
-  (segment (start 160.2105 -28.323) (end 163.0005 -28.323) (width 0.25) (layer F.Cu) (net 41))
-  (segment (start 166.114 -53.973) (end 166.116 -53.975) (width 0.25) (layer F.Cu) (net 41))
-  (segment (start 160.2105 -53.973) (end 166.114 -53.973) (width 0.25) (layer F.Cu) (net 41))
+  (segment (start 165.1254 -41.148) (end 165.1508 -41.1226) (width 0.25) (layer F.Cu) (net 41))
+  (via (at 165.1508 -41.1226) (size 0.8) (drill 0.4) (layers F.Cu B.Cu) (net 41))
+  (segment (start 160.2105 -41.148) (end 165.1254 -41.148) (width 0.25) (layer F.Cu) (net 41))
   (segment (start 168.91 -60.245) (end 168.91 -60.584998) (width 0.25) (layer F.Cu) (net 44))
   (segment (start 168.91 -27.123) (end 171.958 -24.075) (width 0.25) (layer F.Cu) (net 44))
